File: scheme/music_alarm_v0.1/music_alarm.kicad_pcb (KiCad board)
At the start: 2 copper layers, 45 x 25 mm, 42 parts, among them J1 Prog, J2 Alarm, Q1 BSS138, SW1 Button, SW2 5V_IN, SW3 Reset, SW4 USB/DCDC, SW5 RC/PWM, U1 AMS1117-1.2, U2 TPS61221DCK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

Commit message: small: QR code
Change QR code from github to site.
Parts:
- removed the G*** at (137.4, 109.9)
- added G***: LOGO, mine:qr_code, B.Cu at (138.4, 109.7)
